File: ArduinoUnoProtoShield.kicad_pcb (KiCad board)
At the start: 4 copper layers, 68.6 x 53.3 mm, 24 parts

Commit message: auto-backup 2026-07-28 03:26:33
Routing:
- net RESET: track 47.8 -> 54.3 mm
Changed lines of the file:
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@@
+	)
+	(segment
+		(start 3 8)
+		(end 9.5 8)
+		(width 0.4)
+		(layer "F.Cu")
+		(net "RESET")
 	)
 	(segment
